File: Design/H01R0.sch (EAGLE design)
At the start: 27 parts, among them P1 HEXABIT_17.32, Q1 MMBT3904LT1, Q2 MMBT3904LT1, Q3 MMBT3904LT1, U1 STM32G0B1CEU6NUFQFPN48_STM32_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, X1 XTALL_CSTCE8M00G52

Commit message: -Standarize the files and folders
Other:
- note added: "H01R0"
- note added: "H01R0_Backend"
- note added: "H01R0_Frontend"
- note removed: "H01R02"
- note removed: "H01R02_Backend"
- note removed: "H01R02_Frontend"
- note removed: "Obada Albasha"

Commit message: -Improving the Layout Design
Parts:
- D1: value VLMS1300-GS08 -> RED
- FB1: device HEXABITZ_RCLS:FB-TDK_MMZ1608Y300B -> HEXABITZ_RCLS:FB-0603
- U1: value STM32G0B1CEU6NUFQFPN48_STM32_STM -> STM32G0B1CEU6N; device HEXABITZ_ICs:STM32G0B1CEU6NUFQFPN48_STM32_STM -> HEXABITZ_ICs:STM32G0B1CEU6N
Connections:
- net BLED: now also U1.PA6; no longer U1.PB1
- net GLED: now also U1.PB7; no longer U1.PA5
- net GND: no longer U1.PA15, U1.PC13, U1.PC14-OSC32_IN, U1.PD0
- net N$7: now also U1.PB14; no longer U1.PB7
- net RLED: now also U1.PA15; no longer U1.PB13
Other:
- moved on the sheet: D1, JP2, R1, R3
